Commit message: integrated realsense d435 depth camera

File: workspaces/ros2_ws/src/preentend_description/urdf/end_effector/mock.gazebo.xacro (robot description, xacro)
@@ -2,35 +2,5 @@
 <robot xmlns:xacro="http://ros.org/wiki/xacro">
     <xacro:macro name="end_effector_gazebo" params="prefix">
-        <gazebo reference="${prefix}end_effector_base_link">
-            <selfCollide>true</selfCollide>
-        </gazebo>
-        <gazebo reference="${prefix}end_effector_nozzle_1">
-            <selfCollide>true</selfCollide>
-        </gazebo>
-        <gazebo reference="${prefix}end_effector_nozzle_2">
-            <selfCollide>true</selfCollide>
-        </gazebo>
-        <gazebo reference="${prefix}end_effector_nozzle_3">
-            <selfCollide>true</selfCollide>
-        </gazebo>
-        <gazebo reference="${prefix}end_effector_nozzle_4">
-            <selfCollide>true</selfCollide>
-        </gazebo>
-        <gazebo reference="${prefix}end_effector_sensor_1">
-            <selfCollide>true</selfCollide>
-        </gazebo>
-        <gazebo reference="${prefix}end_effector_sensor_2">
-            <selfCollide>true</selfCollide>
-        </gazebo>
-        <gazebo reference="${prefix}end_effector_sensor_3">
-            <selfCollide>true</selfCollide>
-        </gazebo>
-        <gazebo reference="${prefix}end_effector_sensor_4">
-            <selfCollide>true</selfCollide>
-        </gazebo>
-        <gazebo reference="${prefix}end_effector_sensor_5">
-            <selfCollide>true</selfCollide>
-        </gazebo>
-        <gazebo reference="${prefix}end_effector_sensor_6">
+        <gazebo reference="${prefix}end_effector_link">
             <selfCollide>true</selfCollide>
         </gazebo>

File: workspaces/ros2_ws/src/preentend_description/urdf/end_effector/mock_macro.xacro (robot description, xacro)
@@ -1,50 +1,4 @@
 <?xml version="1.0"?>
 <robot xmlns:xacro="http://wiki.ros.org/xacro">
-    <xacro:macro name="end_effector_nozzle_link" params="prefix index">
-        <link name="${prefix}end_effector_nozzle_${index}">
-            <inertial>
-                <mass value="0.0257511" />
-                <origin xyz="-3.71835e-19 -1.24009e-35 0.0389773" rpy="0 -0 0" />
-                <inertia ixx="1.37015e-05" ixy="0" ixz="0" iyy="1.37015e-05" iyz="0"
-                    izz="1.27138e-06" />
-            </inertial>
-            <visual>
-                <geometry>
-                    <mesh
-                        filename="package://preentend_description/meshes/mock_end_effector/end_effector_nozzle.stl" />
-                </geometry>
-                <material name="light_gray" />
-            </visual>
-            <collision>
-                <geometry>
-                    <mesh
-                        filename="package://preentend_description/meshes/mock_end_effector/end_effector_nozzle.stl" />
-                </geometry>
-            </collision>
-        </link>
-    </xacro:macro>
-    <xacro:macro name="end_effector_sensor_link" params="prefix index">
-        <link name="${prefix}end_effector_sensor_${index}">
-            <inertial>
-                <mass value="0.0213081" />
-                <origin xyz="-5.61313e-20 -1.15097e-35 0.0347772" rpy="0 -0 0" />
-                <inertia ixx="1.22295e-05" ixy="0" ixz="0" iyy="1.22295e-05" iyz="0"
-                    izz="9.77537e-07" />
-            </inertial>
-            <visual>
-                <geometry>
-                    <mesh
-                        filename="package://preentend_description/meshes/mock_end_effector/end_effector_sensor.stl" />
-                </geometry>
-                <material name="dark_gray" />
-            </visual>
-            <collision>
-                <geometry>
-                    <mesh
-                        filename="package://preentend_description/meshes/mock_end_effector/end_effector_sensor.stl" />
-                </geometry>
-            </collision>
-        </link>
-    </xacro:macro>
     <xacro:macro name="end_effector"
         params="prefix:=''
@@ -62,106 +16,39 @@
             <child link="${prefix}end_effector_origin" />
         </joint>
-        <link name="${prefix}end_effector_frame" />
-        <joint name="${prefix}end_effector_frame_joint" type="fixed">
-            <origin xyz="0.13125 0 -0.16" rpy="0 0 0"/>
-            <parent link="${prefix}end_effector_origin" />
-            <child link="${prefix}end_effector_frame" />
-        </joint>
-        <link name="${prefix}end_effector_base_link">
+        <link name="${prefix}end_effector_link">
             <inertial>
-                <mass value="1.53208" />
-                <origin xyz="0.118979 0.00187954 -0.118072" rpy="0 -0 0" />
-                <inertia ixx="0.0418325" ixy="-0.000116094" ixz="0.00444694" iyy="0.0397799" iyz="0.000120736" izz="0.00878388" />
+                <mass value="2.20106559" />
+                <origin xyz="0.138 0.012 0.113" rpy="0 0 0" />
+                <inertia
+                    ixx="0.06277067085" ixy="-0.00075440405" ixz="-0.00840932268"
+                    iyy="0.06315719744" iyz="-0.001276814"
+                    izz="0.01607187226" />
             </inertial>
             <visual>
-                <origin xyz="0.02 0 -1.74512e-18" rpy="0 -0 0" />
+                <origin xyz="0 0 0" rpy="0 0 0" />
                 <geometry>
                     <mesh
-                        filename="package://preentend_description/meshes/mock_end_effector/end_effector_base.stl" />
+                        filename="package://preentend_description/meshes/mock_end_effector/visual/end_effector.stl" />
                 </geometry>
                 <material name="gray" />
             </visual>
             <collision>
-                <origin xyz="0.02 0 -1.74512e-18" rpy="0 -0 0" />
+                <origin xyz="0 0 0" rpy="0 0 0" />
                 <geometry>
                     <mesh
-                        filename="package://preentend_description/meshes/mock_end_effector/end_effector_base.stl" />
+                        filename="package://preentend_description/meshes/mock_end_effector/collision/end_effector.stl" />
                 </geometry>
             </collision>
         </link>
-        <joint name="${prefix}end_effector_origin_to_base_joint" type="fixed">
-            <origin xyz="0 0 0" rpy="0 0 0"/>
-            <parent link="${prefix}end_effector_origin"/>
-            <child link="${prefix}end_effector_base_link"/>
+        <joint name="${prefix}end_effector_joint" type="fixed">
+            <origin xyz="0 0 0" rpy="0 0 0" />
+            <parent link="${prefix}end_effector_origin" />
+            <child link="${prefix}end_effector_link" />
         </joint>
-        <xacro:end_effector_nozzle_link prefix="${prefix}" index="1" />
-        <xacro:end_effector_nozzle_link prefix="${prefix}" index="2" />
-        <xacro:end_effector_nozzle_link prefix="${prefix}" index="3" />
-        <xacro:end_effector_nozzle_link prefix="${prefix}" index="4" />
-        <joint name="${prefix}eef_nozzle_j1" type="fixed">
-            <origin xyz="0.135 -0.0475 0.035" rpy="0 1.5708 -0" />
-            <axis xyz="-0 -0 -1" />
-            <parent link="${prefix}end_effector_base_link" />
-            <child link="${prefix}end_effector_nozzle_1" />
-        </joint>
-        <joint name="${prefix}eef_nozzle_j2" type="fixed">
-            <origin xyz="0.135 -0.0475 -0.095" rpy="0 1.5708 -0" />
-            <axis xyz="-0 -0 -1" />
-            <parent link="${prefix}end_effector_base_link" />
-            <child link="${prefix}end_effector_nozzle_2" />
-        </joint>
-        <joint name="${prefix}eef_nozzle_j3" type="fixed">
-            <origin xyz="0.135 -0.0475 -0.225" rpy="0 1.5708 -0" />
-            <axis xyz="-0 -0 -1" />
-            <parent link="${prefix}end_effector_base_link" />
-            <child link="${prefix}end_effector_nozzle_3" />
-        </joint>
-        <joint name="${prefix}eef_nozzle_j4" type="fixed">
-            <origin xyz="0.135 -0.0475 -0.355" rpy="0 1.5708 -0" />
-            <axis xyz="-0 -0 -1" />
-            <parent link="${prefix}end_effector_base_link" />
-            <child link="${prefix}end_effector_nozzle_4" />
-        </joint>
-        <xacro:end_effector_sensor_link prefix="${prefix}" index="1" />
-        <xacro:end_effector_sensor_link prefix="${prefix}" index="2" />
-        <xacro:end_effector_sensor_link prefix="${prefix}" index="3" />
-        <xacro:end_effector_sensor_link prefix="${prefix}" index="4" />
-        <xacro:end_effector_sensor_link prefix="${prefix}" index="5" />
-        <xacro:end_effector_sensor_link prefix="${prefix}" index="6" />
-        <joint name="${prefix}eef_sensor_j1" type="fixed">
-            <origin xyz="0.135 -0.1 0.03875" rpy="0 1.5708 -0" />
-            <axis xyz="-0 -0 -1" />
-            <parent link="${prefix}end_effector_base_link" />
-            <child link="${prefix}end_effector_sensor_1" />
-        </joint>
-        <joint name="${prefix}eef_sensor_j2" type="fixed">
-            <origin xyz="0.135 0.1 0.03875" rpy="0 1.5708 -0" />
-            <axis xyz="-0 -0 -1" />
-            <parent link="${prefix}end_effector_base_link" />
-            <child link="${prefix}end_effector_sensor_2" />
-        </joint>
-        <joint name="${prefix}eef_sensor_j3" type="fixed">
-            <origin xyz="0.135 -0.12 -0.16" rpy="0 1.5708 -0" />
-            <axis xyz="-0 -0 -1" />
-            <parent link="${prefix}end_effector_base_link" />
-            <child link="${prefix}end_effector_sensor_3" />
-        </joint>
-        <joint name="${prefix}eef_sensor_j4" type="fixed">
-            <origin xyz="0.135 0.12 -0.16" rpy="0 1.5708 -0" />
-            <axis xyz="-0 -0 -1" />
-            <parent link="${prefix}end_effector_base_link" />
-            <child link="${prefix}end_effector_sensor_4" />
-        </joint>
-        <joint name="${prefix}eef_sensor_j5" type="fixed">
-            <origin xyz="0.135 -0.1 -0.3625" rpy="0 1.5708 -0" />
-            <axis xyz="-0 -0 -1" />
-            <parent link="${prefix}end_effector_base_link" />
-            <child link="${prefix}end_effector_sensor_5" />
-        </joint>
-        <joint name="${prefix}eef_sensor_j6" type="fixed">
-            <origin xyz="0.135 0.1 -0.3625" rpy="0 1.5708 -0" />
-            <axis xyz="-0 -0 -1" />
-            <parent link="${prefix}end_effector_base_link" />
-            <child link="${prefix}end_effector_sensor_6" />
+        <link name="${prefix}end_effector_frame" />
+        <joint name="${prefix}end_effector_frame_joint" type="fixed">
+            <origin xyz="0.236 0 0.155" rpy="0 0 0" />
+            <parent link="${prefix}end_effector_link" />
+            <child link="${prefix}end_effector_frame" />
         </joint>
     </xacro:macro>

File: workspaces/ros2_ws/src/preentend_description/urdf/robot_macro.xacro (robot description, xacro)
@@ -4,5 +4,5 @@
     <xacro:macro name="robot"
         params="prefix:=''
-        linear_axis_model:='mock' robot_model:='m20_12_23d' end_effector_model:='mock'
+        linear_axis_model:='mock' robot_model:='m20_12_23d' end_effector_model:='mock' camera_model:='realsense'
         parent *origin
         use_gazebo:='false' use_ros2_control:='false' hardware_plugin:='mock_components/GenericSystem'">
@@ -25,4 +25,9 @@
             <origin xyz="0 0 0" rpy="0 0 0" />
         </xacro:end_effector>
+        <xacro:include
+            filename="$(find preentend_description)/urdf/camera/${camera_model}_macro.xacro" />
+        <xacro:camera prefix="${prefix}" parent="${prefix}flange" use_gazebo="${use_gazebo}">
+            <origin xyz="0.226 0 0.431" rpy="0 0 0" />
+        </xacro:camera>
     </xacro:macro>
 </robot>
