Commit message: changed mock end effector cad

File: workspaces/ros2_ws/src/preentend_description/urdf/end_effector/mock_macro.xacro (robot description, xacro)
@@ -62,10 +62,15 @@
             <child link="${prefix}end_effector_origin" />
         </joint>
+        <link name="${prefix}end_effector_frame" />
+        <joint name="${prefix}end_effector_frame_joint" type="fixed">
+            <origin xyz="0.13125 0 -0.16" rpy="0 0 0"/>
+            <parent link="${prefix}end_effector_origin" />
+            <child link="${prefix}end_effector_frame" />
+        </joint>
         <link name="${prefix}end_effector_base_link">
             <inertial>
-                <mass value="1.40889" />
-                <origin xyz="0.104998 2.10691e-17 -0.0977302" rpy="0 -0 0" />
-                <inertia ixx="0.0377398" ixy="0" ixz="0.00470496" iyy="0.0379017" iyz="0"
-                    izz="0.00790301" />
+                <mass value="1.53208" />
+                <origin xyz="0.118979 0.00187954 -0.118072" rpy="0 -0 0" />
+                <inertia ixx="0.0418325" ixy="-0.000116094" ixz="0.00444694" iyy="0.0397799" iyz="0.000120736" izz="0.00878388" />
             </inertial>
             <visual>
@@ -94,8 +99,4 @@
         <xacro:end_effector_nozzle_link prefix="${prefix}" index="3" />
         <xacro:end_effector_nozzle_link prefix="${prefix}" index="4" />
-        <xacro:end_effector_nozzle_link prefix="${prefix}" index="5" />
-        <xacro:end_effector_nozzle_link prefix="${prefix}" index="6" />
-        <xacro:end_effector_nozzle_link prefix="${prefix}" index="7" />
-        <xacro:end_effector_nozzle_link prefix="${prefix}" index="8" />
         <joint name="${prefix}eef_nozzle_j1" type="fixed">
             <origin xyz="0.135 -0.0475 0.035" rpy="0 1.5708 -0" />
@@ -105,5 +106,5 @@
         </joint>
         <joint name="${prefix}eef_nozzle_j2" type="fixed">
-            <origin xyz="0.135 0.0475 0.035" rpy="0 1.5708 -0" />
+            <origin xyz="0.135 -0.0475 -0.095" rpy="0 1.5708 -0" />
             <axis xyz="-0 -0 -1" />
             <parent link="${prefix}end_effector_base_link" />
@@ -111,5 +112,5 @@
         </joint>
         <joint name="${prefix}eef_nozzle_j3" type="fixed">
-            <origin xyz="0.135 -0.0475 -0.095" rpy="0 1.5708 -0" />
+            <origin xyz="0.135 -0.0475 -0.225" rpy="0 1.5708 -0" />
             <axis xyz="-0 -0 -1" />
             <parent link="${prefix}end_effector_base_link" />
@@ -117,32 +118,8 @@
         </joint>
         <joint name="${prefix}eef_nozzle_j4" type="fixed">
-            <origin xyz="0.135 0.0475 -0.095" rpy="0 1.5708 -0" />
+            <origin xyz="0.135 -0.0475 -0.355" rpy="0 1.5708 -0" />
             <axis xyz="-0 -0 -1" />
             <parent link="${prefix}end_effector_base_link" />
             <child link="${prefix}end_effector_nozzle_4" />
-        </joint>
-        <joint name="${prefix}eef_nozzle_j5" type="fixed">
-            <origin xyz="0.135 -0.0475 -0.225" rpy="0 1.5708 -0" />
-            <axis xyz="-0 -0 -1" />
-            <parent link="${prefix}end_effector_base_link" />
-            <child link="${prefix}end_effector_nozzle_5" />
-        </joint>
-        <joint name="${prefix}eef_nozzle_j6" type="fixed">
-            <origin xyz="0.135 0.0475 -0.225" rpy="0 1.5708 -0" />
-            <axis xyz="-0 -0 -1" />
-            <parent link="${prefix}end_effector_base_link" />
-            <child link="${prefix}end_effector_nozzle_6" />
-        </joint>
-        <joint name="${prefix}eef_nozzle_j7" type="fixed">
-            <origin xyz="0.135 -0.0475 -0.355" rpy="0 1.5708 -0" />
-            <axis xyz="-0 -0 -1" />
-            <parent link="${prefix}end_effector_base_link" />
-            <child link="${prefix}end_effector_nozzle_7" />
-        </joint>
-        <joint name="${prefix}eef_nozzle_j8" type="fixed">
-            <origin xyz="0.135 0.0475 -0.355" rpy="0 1.5708 -0" />
-            <axis xyz="-0 -0 -1" />
-            <parent link="${prefix}end_effector_base_link" />
-            <child link="${prefix}end_effector_nozzle_8" />
         </joint>
         <xacro:end_effector_sensor_link prefix="${prefix}" index="1" />
@@ -153,5 +130,5 @@
         <xacro:end_effector_sensor_link prefix="${prefix}" index="6" />
         <joint name="${prefix}eef_sensor_j1" type="fixed">
-            <origin xyz="0.135 -0.04 0.095" rpy="0 1.5708 -0" />
+            <origin xyz="0.135 -0.1 0.03875" rpy="0 1.5708 -0" />
             <axis xyz="-0 -0 -1" />
             <parent link="${prefix}end_effector_base_link" />
@@ -159,5 +136,5 @@
         </joint>
         <joint name="${prefix}eef_sensor_j2" type="fixed">
-            <origin xyz="0.135 0.04 0.095" rpy="0 1.5708 -0" />
+            <origin xyz="0.135 0.1 0.03875" rpy="0 1.5708 -0" />
             <axis xyz="-0 -0 -1" />
             <parent link="${prefix}end_effector_base_link" />
@@ -165,5 +142,5 @@
         </joint>
         <joint name="${prefix}eef_sensor_j3" type="fixed">
-            <origin xyz="0.135 -0.115 -0.16" rpy="0 1.5708 -0" />
+            <origin xyz="0.135 -0.12 -0.16" rpy="0 1.5708 -0" />
             <axis xyz="-0 -0 -1" />
             <parent link="${prefix}end_effector_base_link" />
@@ -171,5 +148,5 @@
         </joint>
         <joint name="${prefix}eef_sensor_j4" type="fixed">
-            <origin xyz="0.135 0.115 -0.16" rpy="0 1.5708 -0" />
+            <origin xyz="0.135 0.12 -0.16" rpy="0 1.5708 -0" />
             <axis xyz="-0 -0 -1" />
             <parent link="${prefix}end_effector_base_link" />
@@ -177,5 +154,5 @@
         </joint>
         <joint name="${prefix}eef_sensor_j5" type="fixed">
-            <origin xyz="0.135 -0.04 -0.415" rpy="0 1.5708 -0" />
+            <origin xyz="0.135 -0.1 -0.3625" rpy="0 1.5708 -0" />
             <axis xyz="-0 -0 -1" />
             <parent link="${prefix}end_effector_base_link" />
@@ -183,5 +160,5 @@
         </joint>
         <joint name="${prefix}eef_sensor_j6" type="fixed">
-            <origin xyz="0.135 0.04 -0.415" rpy="0 1.5708 -0" />
+            <origin xyz="0.135 0.1 -0.3625" rpy="0 1.5708 -0" />
             <axis xyz="-0 -0 -1" />
             <parent link="${prefix}end_effector_base_link" />

File: workspaces/ros2_ws/src/preentend_description/urdf/robot_macro.xacro (robot description, xacro)
@@ -9,12 +9,10 @@
         <xacro:include
             filename="$(find preentend_description)/urdf/linear_axis/${linear_axis_model}_macro.xacro" />
-        <xacro:include
-            filename="$(find preentend_description)/urdf/robot/${robot_model}_macro.xacro" />
-        <xacro:include
-            filename="$(find preentend_description)/urdf/end_effector/${end_effector_model}_macro.xacro" />
         <xacro:linear_axis prefix="${prefix}" parent="${parent}" use_gazebo="${use_gazebo}"
             use_ros2_control="${use_ros2_control}" hardware_plugin="${hardware_plugin}">
             <xacro:insert_block name="origin" />
         </xacro:linear_axis>
+        <xacro:include
+            filename="$(find preentend_description)/urdf/robot/${robot_model}_macro.xacro" />
         <xacro:robot_arm prefix="${prefix}" parent="${prefix}linear_axis_carrier_mount"
             use_gazebo="${use_gazebo}"
@@ -22,4 +20,6 @@
             <origin xyz="0 0 0" rpy="0 0 0" />
         </xacro:robot_arm>
+        <xacro:include
+            filename="$(find preentend_description)/urdf/end_effector/${end_effector_model}_macro.xacro" />
         <xacro:end_effector prefix="${prefix}" parent="${prefix}flange" use_gazebo="${use_gazebo}">
             <origin xyz="0 0 0" rpy="0 0 0" />

Commit message: minor visual changes. logic untouched

File: workspaces/ros2_ws/src/preentend_description/urdf/end_effector/mock_macro.xacro (robot description, xacro)
@@ -46,9 +46,9 @@
             <child link="${prefix}end_effector_link" />
         </joint>
-        <link name="${prefix}end_effector_frame" />
-        <joint name="${prefix}end_effector_frame_joint" type="fixed">
+        <link name="${prefix}tcp" />
+        <joint name="${prefix}tcp_joint" type="fixed">
             <origin xyz="0.236 0 0.155" rpy="0 0 0" />
             <parent link="${prefix}end_effector_link" />
-            <child link="${prefix}end_effector_frame" />
+            <child link="${prefix}tcp" />
         </joint>
     </xacro:macro>
